File: base-module.kicad_pcb (KiCad board)
At the start: 4 copper layers, 100 x 100 mm, 166 parts, among them J200 09031967921, J800 USB_C_Receptacle_USB2.0_16P, Q700 MMST3904, U100 W25Q128, U300 TPS563200, U301 TPS563200, U302 CH334P, U401 TPD2E2U06DCK, U402 TPD2E2U06DCK, U403 STM32H562VGTx, U500 TJA1044GTK_3Z, U600 TJA1044GTK_3Z, U700 STM32F103CBTx, U801 FSUSB42UMX, X300 Q13FC1350000400, Y400 ASE-xxxMHz, Y700 8 MHz, Y900 12Mhz

Commit message: [#8] Fix LEDs resistors values
Parts:
- removed R400: 1.2kΩ, PCM_JLCPCB:R_0402
- removed R408: 220Ω, PCM_JLCPCB:R_0402
- removed R409: 100Ω, PCM_JLCPCB:R_0402
- added R414: 220Ω, PCM_JLCPCB:R_0402, F.Cu at (114.5, 61.2)
- added R415: 220Ω, PCM_JLCPCB:R_0402, F.Cu at (115.3, 61.2)
- added R416: 220Ω, PCM_JLCPCB:R_0402, F.Cu at (113.5, 61.2)
